Commit message: minor fixes, here and there

File: bumperbot_description/urdf/camera.xacro (robot description, xacro)
@@ -27,5 +27,5 @@
         <parent link="foundation" />
         <child link="cam_base_link" />
-        <origin xyz="2 2 0" rpy="0 0 0" />
+        <origin xyz="0 -1 0" rpy="0 0 0" />
         <axis xyz="0 0 0" />
     </joint>
@@ -62,11 +62,4 @@
         </joint>
     </xacro:macro>
-    <xacro:macro name="camera_optical_link" params="name parent child">
-        <joint name="${name}" type="fixed">
-            <parent link="${parent}" />
-            <child link="${child}" />
-            <origin xyz="0 0 0" rpy="-1.5708 0 1.5708" />
-        </joint>
-    </xacro:macro>
     <xacro:macro name="camera_gazebo_ref" params="link_name camera_name">
         <gazebo reference="${link_name}">
@@ -79,5 +72,6 @@
                 <camera>
                     <camera_info_topic>${camera_name}/camera_info</camera_info_topic>
-                    <horizontal_fov>1.047</horizontal_fov>
+                    <!-- In radians, so approximately 150 degrees-->
+                    <horizontal_fov>2.61799</horizontal_fov>
                     <image>
                         <width>640</width>
@@ -87,5 +81,5 @@
                     <clip>
                         <near>0.05</near>
-                        <far>8.0</far>
+                        <far>100.0</far>
                     </clip>
                 </camera>
@@ -107,10 +101,5 @@
         xyz="-0.23575 0 3.391"
         rpy="0.15764 -0.17851 -0.028217" />
-    <xacro:camera_optical_link
-        name="camera_optical_link_north"
-        parent="camera_link_north"
-        child="camera_link_optical_north" />
-    <link name="camera_link_optical_north" />
-    <xacro:camera_gazebo_ref link_name="camera_link_optical_north" camera_name="camera_north" />
+    <xacro:camera_gazebo_ref link_name="camera_link_north" camera_name="camera_north" />
     <xacro:camera_link
         name="camera_link_east"
@@ -125,10 +114,5 @@
         xyz="0 -0.23575 3.511"
         rpy="-0.15257 0.18285 -1.5708" />
-    <xacro:camera_optical_link
-        name="camera_optical_link_east"
-        parent="camera_link_east"
-        child="camera_link_optical_east" />
-    <link name="camera_link_optical_east" />
-    <xacro:camera_gazebo_ref link_name="camera_link_optical_east" camera_name="camera_east" />
+    <xacro:camera_gazebo_ref link_name="camera_link_east" camera_name="camera_east" />
     <xacro:camera_link
         name="camera_link_south"
@@ -143,10 +127,5 @@
         xyz="0.23575 0 3.391"
         rpy="0.15257 -0.18285 3.1416" />
-    <xacro:camera_optical_link
-        name="camera_optical_link_south"
-        parent="camera_link_south"
-        child="camera_link_optical_south" />
-    <link name="camera_link_optical_south" />
-    <xacro:camera_gazebo_ref link_name="camera_link_optical_south" camera_name="camera_south" />
+    <xacro:camera_gazebo_ref link_name="camera_link_south" camera_name="camera_south" />
     <xacro:camera_link
         name="camera_link_west"
@@ -161,9 +140,4 @@
         xyz="0 0.23575 3.511"
         rpy="-0.15257 0.18285 1.5708" />
-    <xacro:camera_optical_link
-        name="camera_optical_link_west"
-        parent="camera_link_west"
-        child="camera_link_optical_west" />
-    <link name="camera_link_optical_west" />
-    <xacro:camera_gazebo_ref link_name="camera_link_optical_west" camera_name="camera_west" />
+    <xacro:camera_gazebo_ref link_name="camera_link_west" camera_name="camera_west" />
 </robot>

Commit message: Cameras set up, thief set up

File: bumperbot_description/urdf/camera.xacro (robot description, xacro)
@@ -62,4 +62,14 @@
         </joint>
     </xacro:macro>
+    <xacro:macro name="camera_optical_link_joint" params="name parent child">
+        <joint name="${name}" type="fixed">
+            <parent link="${parent}" />
+            <child link="${child}" />
+            <origin xyz="0 0 0" rpy="0 0 ${pi}" />
+        </joint>
+    </xacro:macro>
+    <xacro:macro name="camera_optical_link" params="name">
+        <link name="${name}"/>
+    </xacro:macro>
     <xacro:macro name="camera_gazebo_ref" params="link_name camera_name">
         <gazebo reference="${link_name}">
@@ -101,5 +111,11 @@
         xyz="-0.23575 0 3.391"
         rpy="0.15764 -0.17851 -0.028217" />
-    <xacro:camera_gazebo_ref link_name="camera_link_north" camera_name="camera_north" />
+    <xacro:camera_optical_link
+        name="camera_optical_link_north"/>
+    <xacro:camera_optical_link_joint
+        name="camera_optical_link_joint_north"
+        parent="camera_link_north"
+        child="camera_optical_link_north"/>
+    <xacro:camera_gazebo_ref link_name="camera_optical_link_north" camera_name="camera_north" />
     <xacro:camera_link
         name="camera_link_east"
@@ -127,5 +143,11 @@
         xyz="0.23575 0 3.391"
         rpy="0.15257 -0.18285 3.1416" />
-    <xacro:camera_gazebo_ref link_name="camera_link_south" camera_name="camera_south" />
+         <xacro:camera_optical_link
+        name="camera_optical_link_south"/>
+    <xacro:camera_optical_link_joint
+        name="camera_optical_link_joint_south"
+        parent="camera_link_south"
+        child="camera_optical_link_south"/>
+    <xacro:camera_gazebo_ref link_name="camera_optical_link_south" camera_name="camera_south" />
     <xacro:camera_link
         name="camera_link_west"
