Commit message: ros2 control added

File: bumperbot_description/urdf/bumperbot.urdf.xacro (robot description, xacro)
@@ -1,5 +1,6 @@
 <?xml version="1.0" encoding="UTF-8"?>
 <robot xmlns:xacro="http://www.ros.org/wiki/xacro" name="bumperbot">
-    <xacro:include filename="$(find bumoerbot_description)/urdf/bumperbot_gazebo.xacro" />
+    <xacro:include filename="$(find bumperbot_description)/urdf/bumperbot_gazebo.xacro" />
+    <xacro:include filename="$(find bumperbot_description)/urdf/bumperbot_ros2_control.xacro" />
     <link name="base_footprint" />
     <link name="base_link">

File: bumperbot_description/urdf/bumperbot_gazebo.xacro (robot description, xacro)
@@ -1,41 +1,62 @@
 <?xml version="1.0" encoding="UTF-8"?>
 <robot name="bumperbot" xmlns:xacro="http://www.ros.org/wiki/xacro">
+    <transmission name="wheel_right_transmission">
+        <plugin>transmission_interface/SimpleTransmission</plugin>
+        <actuator name="wheel_right_motor" role="actuator_right" />
+        <joint name="wheel_right_joint" role="joint_right">
+            <mechanical_reduction>1.0</mechanical_reduction>
+        </joint>
+    </transmission>
+    <transmission name="wheel_left_transmission">
+        <plugin>transmission_interface/SimpleTransmission</plugin>
+        <actuator name="wheel_left_motor" role="actuator_left" />
+        <joint name="wheel_left_joint" role="joint_left">
+            <mechanical_reduction>1.0</mechanical_reduction>
+        </joint>
+    </transmission>
     <gazebo reference="wheel_right_link">
         <!-- friction coeeficients-->
-         <mu1>100000000000000.0</mu1>
-         <mu2>100000000000000.0</mu2>
-         <kp>1000000000000.0</kp>
-         <kd>10.0</kd>
-         <minDeoth>0.001</minDeoth>
-         <maxVel>0.1</maxVel>
+        <mu1>100000000000000.0</mu1>
+        <mu2>100000000000000.0</mu2>
+        <kp>1000000000000.0</kp>
+        <kd>10.0</kd>
+        <minDeoth>0.001</minDeoth>
+        <maxVel>0.1</maxVel>
         <fdir>1 0 0</fdir>
     </gazebo>
     <gazebo reference="wheel_left_link">
         <!-- friction coeeficients-->
-         <mu1>100000000000000.0</mu1>
-         <mu2>100000000000000.0</mu2>
-         <kp>1000000000000.0</kp>
-         <kd>10.0</kd>
-         <minDeoth>0.001</minDeoth>
-         <maxVel>0.1</maxVel>
+        <mu1>100000000000000.0</mu1>
+        <mu2>100000000000000.0</mu2>
+        <kp>1000000000000.0</kp>
+        <kd>10.0</kd>
+        <minDeoth>0.001</minDeoth>
+        <maxVel>0.1</maxVel>
         <fdir>1 0 0</fdir>
     </gazebo>
     <gazebo reference="caster_front_link">
         <!-- friction coeeficients-->
-         <mu1>0.1</mu1>
-         <mu2>0.1</mu2>
-         <kp>1000000.0</kp>
-         <kd>100.0</kd>
-         <minDeoth>0.001</minDeoth>
-         <maxVel>0.1</maxVel>
+        <mu1>0.1</mu1>
+        <mu2>0.1</mu2>
+        <kp>1000000.0</kp>
+        <kd>100.0</kd>
+        <minDeoth>0.001</minDeoth>
+        <maxVel>0.1</maxVel>
     </gazebo>
     <gazebo reference="caster_rear_link">
         <!-- friction coeeficients-->
-         <mu1>0.1</mu1>
-         <mu2>0.1</mu2>
-         <kp>1000000.0</kp>
-         <kd>100.0</kd>
-         <minDeoth>0.001</minDeoth>
-         <maxVel>0.1</maxVel>
+        <mu1>0.1</mu1>
+        <mu2>0.1</mu2>
+        <kp>1000000.0</kp>
+        <kd>100.0</kd>
+        <minDeoth>0.001</minDeoth>
+        <maxVel>0.1</maxVel>
+    </gazebo>
+    <gazebo>
+        <plugin filename="libgazebo_ros2_control.so" name="gazebo_ros2_control">
+            <robot_param>robot_description</robot_param>
+            <robot_param_node>robot_state_publisher</robot_param_node>
+            <parameters>$(find bumperbot_controller)/config/bumperbot_controllers.yaml</parameters>
+        </plugin>
     </gazebo>
 </robot>

Commit message: implemented a kalman filter

File: bumperbot_description/urdf/bumperbot.urdf.xacro (robot description, xacro)
@@ -1,5 +1,5 @@
 <?xml version="1.0" encoding="UTF-8"?>
 <robot xmlns:xacro="http://www.ros.org/wiki/xacro" name="bumperbot">
-    <xacro:arg name="is_humble" default="false"/>
+    <xacro:arg name="is_humble" default="false" />
     <xacro:include filename="$(find bumperbot_description)/urdf/bumperbot_gazebo.xacro" />
     <xacro:include filename="$(find bumperbot_description)/urdf/bumperbot_ros2_control.xacro" />
@@ -150,3 +150,31 @@
         <origin xyz="-0.03 0.03 0.078" rpy="1.57 0 0" />
     </joint> -->
+    <link name="imu_link">
+        <inertial>
+            <origin xyz="-0.00552433659106688 0.000168210391520346 0.000514000497342681" rpy="0 0 0" />
+            <mass value="0.000528415362211671" />
+            <inertia ixx="1.46176048428261E-08" ixy="1.40015117949421E-10"
+                ixz="-1.99633872937403E-12"
+                iyy="8.59662482954888E-09" iyz="7.52375112767959E-12"
+                izz="2.30279421279312E-08" />
+        </inertial>
+        <visual>
+            <origin xyz="0 0 0" rpy="0 0 0" />
+            <geometry>
+                <mesh filename="package://bumperbot_description/meshes/imu_link.STL" />
+            </geometry>
+        </visual>
+        <collision>
+            <origin xyz="0 0 0" rpy="0 0 0" />
+            <geometry>
+                <mesh filename="package://bumperbot_description/meshes/imu_link.STL" />
+            </geometry>
+        </collision>
+    </link>
+    <joint name="imu_joint" type="fixed">
+        <origin xyz="0 0 0.0698986241758014" rpy="0 0 0" />
+        <parent link="base_link" />
+        <child link="imu_link" />
+        <axis xyz="0 0 0" />
+    </joint>
 </robot>

File: bumperbot_description/urdf/bumperbot_gazebo.xacro (robot description, xacro)
@@ -62,8 +62,61 @@
         </xacro:if>
         <xacro:unless value="$(arg is_humble)">
-            <plugin filename="gz_ros2_control-system" name="gz_ros2_control::GazeboSimROS2ControlPlugin">
+            <plugin filename="gz_ros2_control-system"
+                name="gz_ros2_control::GazeboSimROS2ControlPlugin">
                 <parameters>$(find bumperbot_controller)/config/bumperbot_controllers.yaml</parameters>
+            </plugin>
+            <plugin filename="gz-sim-imu-system" name="gz::sim::systems::Imu">
             </plugin>
         </xacro:unless>
     </gazebo>
+    <gazebo reference="imu_link">
+        <sensor name="imu" type="imu">
+            <always_on>true</always_on>
+            <update_rate>100</update_rate>
+            <gz_frame_id>imu_link</gz_frame_id>
+            <topic>imu</topic>
+            <imu>
+                <angular_velocity>
+                    <x>
+                        <noise type="gaussian">
+                            <mean>0.0</mean>
+                            <stddev>2e-4</stddev>
+                        </noise>
+                    </x>
+                    <y>
+                        <noise type="gaussian">
+                            <mean>0.0</mean>
+                            <stddev>2e-4</stddev>
+                        </noise>
+                    </y>
+                    <z>
+                        <noise type="gaussian">
+                            <mean>0.0</mean>
+                            <stddev>2e-4</stddev>
+                        </noise>
+                    </z>
+                </angular_velocity>
+                <linear_velocity>
+                    <x>
+                        <noise type="gaussian">
+                            <mean>0.0</mean>
+                            <stddev>1.7e-2</stddev>
+                        </noise>
+                    </x>
+                    <y>
+                        <noise type="gaussian">
+                            <mean>0.0</mean>
+                            <stddev>1.7e-2</stddev>
+                        </noise>
+                    </y>
+                    <z>
+                        <noise type="gaussian">
+                            <mean>0.0</mean>
+                            <stddev>1.7e-2</stddev>
+                        </noise>
+                    </z>
+                </linear_velocity>
+            </imu>
+        </sensor>
+    </gazebo>
 </robot>

Commit message: updates

File: bumperbot_description/urdf/bumperbot.urdf.xacro (robot description, xacro)
@@ -1,6 +1,13 @@
-<?xml version="1.0" encoding="UTF-8"?>
-<robot xmlns:xacro="http://www.ros.org/wiki/xacro" name="bumperbot">
+<?xml version="1.0"?>
+<robot name="bumperbot" xmlns:xacro="http://ros.org/wiki/xacro">
+    <!-- Start GZ or Ignition depending on ROS 2 Version -->
+    <xacro:arg name="is_ignition" default="true" />
+    <!-- Load Simulated or Real Hardware Interfaces -->
+    <xacro:arg name="is_sim" default="true" />
+    <!-- ROS2 Humble or Jazzy-->
     <xacro:arg name="is_humble" default="false" />
+    <!-- Include Gazebo Parameters -->
     <xacro:include filename="$(find bumperbot_description)/urdf/bumperbot_gazebo.xacro" />
+    <!-- Include ros2_control Plugins -->
     <xacro:include filename="$(find bumperbot_description)/urdf/bumperbot_ros2_control.xacro" />
     <link name="base_footprint" />
@@ -10,17 +17,19 @@
             <mass value="8.2573504e-01" />
             <inertia ixx="2.2124416e-02" ixy="-1.2294101e-04" ixz="3.4938785e-04"
-                iyy="2.1193702e-02" iyz="-5.0120904e-05" izz="2.0064271e-02" />
-        </inertial>
-        <visual>
+                iyy="2.1193702e-02" iyz="-5.0120904e-05"
+                izz="2.0064271e-02" />
+        </inertial>
+        <visual>
+            <origin xyz="0 0 0" rpy="0 0 0" />
             <geometry>
                 <mesh filename="package://bumperbot_description/meshes/base_link.STL" />
             </geometry>
-            <origin rpy="0 0 0" xyz="0 0 0" />
-        </visual>
-        <collision>
+            <material name="black" />
+        </visual>
+        <collision>
+            <origin xyz="0 0 0" rpy="0 0 0" />
             <geometry>
                 <mesh filename="package://bumperbot_description/meshes/base_link.STL" />
             </geometry>
-            <origin rpy="0 0 0" xyz="0 0 0" />
         </collision>
     </link>
@@ -35,12 +44,14 @@
             <mass value="0.0530086090966721" />
             <inertia ixx="1.88176298336665E-05" ixy="-4.8444933029987E-10"
-                ixz="1.88163708851143E-08" iyy="3.11510738647764E-05" iyz="-6.93560663069607E-11"
+                ixz="1.88163708851143E-08"
+                iyy="3.11510738647764E-05" iyz="-6.93560663069607E-11"
                 izz="1.8801969558182E-05" />
         </inertial>
         <visual>
-            <origin rpy="1.57 0 0" xyz="0 0 0" />
+            <origin xyz="0 0 0" rpy="1.57 0 0" />
             <geometry>
                 <mesh filename="package://bumperbot_description/meshes/wheel_right_link.STL" />
             </geometry>
+            <material name="blue" />
         </visual>
         <collision>
@@ -52,25 +63,28 @@
     </link>
     <joint name="wheel_right_joint" type="continuous">
+        <origin xyz="0 -0.0701101849418637 0" rpy="0 0 0" />
         <parent link="base_link" />
         <child link="wheel_right_link" />
-        <origin xyz="0 -0.07 0" rpy="0 0 0" />
         <axis xyz="0 1 0" />
     </joint>
-    <link name="wheel_left_link">
-        <inertial>
-            <origin xyz="0 -0.014 0" rpy="0 0 0" />
-            <mass value="0.0530086090966721" />
-            <inertia ixx="1.88176298336665E-05" ixy="-4.8444933029987E-10"
-                ixz="1.88163708851143E-08" iyy="3.11510738647764E-05" iyz="-6.93560663069607E-11"
-                izz="1.8801969558182E-05" />
-        </inertial>
-        <visual>
-            <origin rpy="-1.57 0 0" xyz="0 0 0" />
+    <link
+        name="wheel_left_link">
+        <inertial>
+            <origin xyz="0 0.014 0" rpy="0 0 0" />
+            <mass value="0.0530086043217644" />
+            <inertia ixx="1.8792911368909E-05" ixy="3.31256392204584E-10"
+                ixz="-1.14082001662767E-08"
+                iyy="3.11510738759073E-05" iyz="-3.60499245082192E-10"
+                izz="1.88266886146847E-05" />
+        </inertial>
+        <visual>
+            <origin xyz="0 0 0" rpy="-1.57 0 0" />
             <geometry>
                 <mesh filename="package://bumperbot_description/meshes/wheel_left_link.STL" />
             </geometry>
-        </visual>
-        <collision>
-            <origin xyz="0 0.015 0" rpy="1.57 0 0" />
+            <material name="blue" />
+        </visual>
+        <collision>
+            <origin xyz="0 0.015 0" rpy="-1.57 0 0" />
             <geometry>
                 <sphere radius="0.033" />
@@ -79,7 +93,7 @@
     </link>
     <joint name="wheel_left_joint" type="continuous">
+        <origin xyz="0 0.0701101849418642 0" rpy="0 0 0" />
         <parent link="base_link" />
         <child link="wheel_left_link" />
-        <origin xyz="0 0.07 0" rpy="0 0 0" />
         <axis xyz="0 1 0" />
     </joint>
@@ -89,5 +103,6 @@
             <mass value="1.44379265037903E-06" />
             <inertia ixx="7.23075276010246E-11" ixy="-6.10956883467859E-16"
-                ixz="2.22849693525031E-15" iyy="3.8713793085917E-11" iyz="2.93909858781952E-15"
+                ixz="2.22849693525031E-15"
+                iyy="3.8713793085917E-11" iyz="2.93909858781952E-15"
                 izz="1.00967486676306E-10" />
         </inertial>
@@ -97,4 +112,5 @@
                 <mesh filename="package://bumperbot_description/meshes/caster_front_link.STL" />
             </geometry>
+            <material name="silver" />
         </visual>
         <collision>
@@ -106,7 +122,8 @@
     </link>
     <joint name="caster_front_joint" type="fixed">
+        <origin xyz="0.04755 0 -0.0275" rpy="0 0 0" />
         <parent link="base_link" />
         <child link="caster_front_link" />
-        <origin xyz="0.04755 0 -0.0275" rpy="0 0 0" />
+        <axis xyz="0 0 0" />
     </joint>
     <link name="caster_rear_link">
@@ -115,5 +132,6 @@
             <mass value="1.44379265037902E-06" />
             <inertia ixx="7.23075276010246E-11" ixy="-6.10956872363424E-16"
-                ixz="2.22849693527207E-15" iyy="3.87137930859167E-11" iyz="2.939098587861E-15"
+                ixz="2.22849693527207E-15"
+                iyy="3.87137930859167E-11" iyz="2.939098587861E-15"
                 izz="1.00967486676306E-10" />
         </inertial>
@@ -123,4 +141,5 @@
                 <mesh filename="package://bumperbot_description/meshes/caster_rear_link.STL" />
             </geometry>
+            <material name="silver" />
         </visual>
         <collision>
@@ -132,22 +151,9 @@
     </link>
     <joint name="caster_rear_joint" type="fixed">
+        <origin xyz="-0.04755 0 -0.0275" rpy="0 0 0" />
         <parent link="base_link" />
         <child link="caster_rear_link" />
-        <origin xyz="-0.04755 0 -0.0275" rpy="0 0 0" />
-    </joint>
-    <!-- Assignment -->
-    <!-- <link name="can_link">
-        <visual>
-            <origin rpy="0 0 0" xyz="0 0 0" />
-            <geometry>
-                <mesh filename="package://bumperbot_description/meshes/can.STL" />
-            </geometry>
-        </visual>
-    </link>
-    <joint name="can_joint" type="fixed">
-        <parent link="base_link" />
-        <child link="can_link" />
-        <origin xyz="-0.03 0.03 0.078" rpy="1.57 0 0" />
-    </joint> -->
+        <axis xyz="0 0 0" />
+    </joint>
     <link name="imu_link">
         <inertial>
@@ -164,4 +170,5 @@
                 <mesh filename="package://bumperbot_description/meshes/imu_link.STL" />
             </geometry>
+            <material name="blue" />
         </visual>
         <collision>
@@ -178,3 +185,44 @@
         <axis xyz="0 0 0" />
     </joint>
+    <link name="laser_link">
+        <inertial>
+            <origin xyz="-0.011945780406062 -0.000381929217680526 -0.0170649378129477" rpy="0 0 0" />
+            <mass value="0.073084435549317" />
+            <inertia ixx="1.96074931730795E-05" ixy="-3.62091076640009E-07"
+                ixz="4.28230084046735E-07"
+                iyy="2.40983835136327E-05" iyz="1.50180909250652E-08"
+                izz="4.14184164228595E-05" />
+        </inertial>
+        <visual>
+            <origin xyz="0 0 0" rpy="0 0 0" />
+            <geometry>
+                <mesh filename="package://bumperbot_description/meshes/laser_link.STL" />
+            </geometry>
+            <material name="dark_grey" />
+        </visual>
+        <collision>
+            <origin xyz="0 0 0" rpy="0 0 0" />
+            <geometry>
+                <mesh filename="package://bumperbot_description/meshes/laser_link.STL" />
+            </geometry>
+        </collision>
+    </link>
+    <joint name="laser_joint" type="fixed">
+        <origin xyz="-0.0050526 -0.0023221 0.1208" rpy="0 0 3.14" />
+        <parent link="base_link" />
+        <child link="laser_link" />
+        <axis xyz="0 0 0" />
+    </joint>
+    <material name="blue">
+        <color rgba="0 0 1 1" />
+    </material>
+    <material name="black">
+        <color rgba="0 0 0 1" />
+    </material>
+    <material name="silver">
+        <color rgba="0.79 0.82 0.93 1" />
+    </material>
+    <material name="dark_grey">
+        <color rgba="0.3 0.3 0.3 1" />
+    </material>
 </robot>

File: bumperbot_description/urdf/bumperbot_gazebo.xacro (robot description, xacro)
@@ -68,4 +68,7 @@
             <plugin filename="gz-sim-imu-system" name="gz::sim::systems::Imu">
             </plugin>
+            <plugin filename="gz-sim-sensors-system" name="gz::sim::systems::Sensors">
+                <render_engine>ogre2</render_engine>
+            </plugin>
         </xacro:unless>
     </gazebo>
@@ -120,3 +123,32 @@
         </sensor>
     </gazebo>
+    <gazebo reference="laser_link">
+        <sensor name="lidar" type="gpu_lidar">
+          <always_on>true</always_on>
+          <visualize>true</visualize>
+          <topic>scan</topic>
+          <update_rate>5</update_rate>
+          <gz_frame_id>laser_link</gz_frame_id>
+          <lidar>
+            <scan>
+              <horizontal>
+                <samples>360</samples>
+                <resolution>1.00000</resolution>
+                <min_angle>0.000000</min_angle>
+                <max_angle>6.280000</max_angle>
+              </horizontal>
+            </scan>
+            <range>
+              <min>0.120000</min>
+              <max>12.0</max>
+              <resolution>0.02</resolution>
+            </range>
+            <noise>
+              <type>gaussian</type>
+              <mean>0.0</mean>
+              <stddev>0.01</stddev>
+            </noise>
+          </lidar>
+        </sensor>
+      </gazebo>
 </robot>

Commit message: cameras working

File: bumperbot_description/urdf/bumperbot.urdf.xacro (robot description, xacro)
@@ -12,5 +12,5 @@
     <xacro:include filename="$(find bumperbot_description)/urdf/bumperbot_ros2_control.xacro" />
     <!-- Include Camera -->
-    <xacro:include filename="$(find bumperbot_description)/urdf/camera.xacro"/>
+    <!-- <xacro:include filename="$(find bumperbot_description)/urdf/camera.xacro" /> -->
     <link name="base_footprint" />
     <link name="base_link">

File: bumperbot_description/urdf/camera.xacro (robot description, xacro)
@@ -1,4 +1,5 @@
 <?xml version="1.0" encoding="UTF-8"?>
-<robot xmlns:xacro="http://www.ros.org/wiki/xacro" name="robot_name">
+<robot xmlns:xacro="http://www.ros.org/wiki/xacro" name="camera_stand">
+    <link name="foundation" />
     <!-- Base Link -->
     <link name="cam_base_link">
@@ -15,7 +16,14 @@
             </geometry>
         </collision>
+        <inertial>
+            <origin xyz="0 0 0" rpy="0.0 0.0 0.0" />
+            <mass value="1" />
+            <inertia ixx="1" ixy="0" ixz="0"
+                iyy="1" iyz="0"
+                izz="1" />
+        </inertial>
     </link>
-    <joint name="foundation_!" type="fixed">
-        <parent link="base_footprint" />
+    <joint name="fixation" type="fixed">
+        <parent link="foundation" />
         <child link="cam_base_link" />
         <origin xyz="2 2 0" rpy="0 0 0" />
@@ -37,4 +45,11 @@
                 </geometry>
             </collision>
+            <inertial>
+                <origin xyz="0 0 0" rpy="0.0 0.0 0.0" />
+                <mass value="1" />
+                <inertia ixx="1" ixy="0" ixz="0"
+                    iyy="1" iyz="0"
+                    izz="1" />
+            </inertial>
         </link>
     </xacro:macro>
@@ -56,11 +71,12 @@
     <xacro:macro name="camera_gazebo_ref" params="link_name camera_name">
         <gazebo reference="${link_name}">
-            <gz_frame_id>${link_name}</gz_frame_id>
-            <always_on>true</always_on>
-            <visualize>true</visualize>
-            <update_rate>5</update_rate>
             <sensor name="${camera_name}" type="camera">
+                <gz_frame_id>${link_name}</gz_frame_id>
+                <always_on>true</always_on>
+                <visualize>true</visualize>
+                <update_rate>10</update_rate>
                 <pose>0 0 0 0 0 0</pose>
                 <camera>
+                    <camera_info_topic>${camera_name}/camera_info</camera_info_topic>
                     <horizontal_fov>1.047</horizontal_fov>
                     <image>
@@ -74,4 +90,5 @@
                     </clip>
                 </camera>
+                <topic>${camera_name}/image_raw</topic>
             </sensor>
         </gazebo>
