Commit message: gogo

File: bumperbot_description/urdf/bumperbot.urdf.xacro (robot description, xacro)
@@ -216,4 +216,30 @@
         <axis xyz="0 0 0" />
     </joint>
+    <link name="cam_link_bumperbot">
+        <visual>
+            <geometry>
+                <box size="0.01 0.01 0.01" />
+            </geometry>
+            <material name="LightGrey">
+                <color rgba="0.7 0.7 0.7 1.0"/>
+            </material>
+        </visual>
+        <collision>
+            <geometry>
+                <box size="0.01 0.01 0.01" />
+            </geometry>
+        </collision>
+        <inertial>
+            <mass value="0.0"/>
+            <origin xyz="0.0 0.0 0.0" rpy="0.0 0.0 0.0"/>
+            <inertia ixx="0.0" ixy="0.0" ixz="0.0" iyy="0.0" iyz="0.0" izz="0.0"/>
+        </inertial>
+    </link>
+    <joint name="cam_bumperbot" type="fixed">
+        <parent link="base_link"/>
+        <child link="cam_link_bumperbot"/>
+         <origin xyz="0.064 0 0.08498986241758014" rpy="0 0 0" />
+        <axis xyz="0 0 0"/>
+    </joint>
     <material name="blue">
         <color rgba="0 0 1 1" />

File: bumperbot_description/urdf/bumperbot_gazebo.xacro (robot description, xacro)
@@ -152,3 +152,27 @@
         </sensor>
     </gazebo>
+    <gazebo reference="cam_link_bumperbot">
+        <sensor name="bumperbot_camera" type="camera">
+            <gz_frame_id>cam_link_bumperbot</gz_frame_id>
+            <always_on>true</always_on>
+            <visualize>true</visualize>
+            <update_rate>10</update_rate>
+            <pose>0 0 0 0 0 0</pose>
+            <camera>
+                <camera_info_topic>bumperbot_camera/camera_info</camera_info_topic>
+                <!-- In radians, so approximately 90 degrees-->
+                <horizontal_fov>1.571</horizontal_fov>
+                <image>
+                    <width>640</width>
+                    <height>480</height>
+                    <format>R8G8B8</format>
+                </image>
+                <clip>
+                    <near>0.05</near>
+                    <far>100.0</far>
+                </clip>
+            </camera>
+            <topic>bumperbot_camera/image_raw</topic>
+        </sensor>
+    </gazebo>
 </robot>

File: bumperbot_description/urdf/camera.xacro (robot description, xacro)
@@ -9,4 +9,5 @@
                 <mesh filename="package://bumperbot_description/meshes/cam_base_link.STL" />
             </geometry>
+            <material name="black"/>
         </visual>
         <collision>
@@ -38,4 +39,5 @@
                     <mesh filename="${filename}" />
                 </geometry>
+                <material name="blue"/>
             </visual>
             <collision>
@@ -98,4 +100,33 @@
         </gazebo>
     </xacro:macro>
+    <!-- Define Ball -->
+    <!-- <link name="ball">
+        <visual>
+            <geometry>
+                <sphere radius="0."/>
+            </geometry>
+            <material name="yellow">
+                <color rgba="1 1 0 1"/>
+            </material>
+        </visual>
+        <collision>
+            <geometry>
+                <sphere radius="0.1"/>
+            </geometry>
+        </collision>
+        <inertial>
+            <mass value="0.1"/>
+            <origin xyz="0 0 0"/>
+            <inertia ixx="0.0001" ixy="0" ixz="0"
+                iyy="0.0001" iyz="0"
+                izz="0.0001"/>
+        </inertial>
+    </link>
+    <joint name="ball_location" type="fixed">
+        <parent link="foundation"/>
+        <child link="ball"/>
+        <origin xyz="1 0 0" rpy="0 0 0"/>
+        <axis xyz="0 0 0"/>
+    </joint> -->
     <!-- Define Cameras -->
     <xacro:camera_link
@@ -163,3 +194,15 @@
         rpy="-0.15257 0.18285 1.5708" />
     <xacro:camera_gazebo_ref link_name="camera_link_west" camera_name="camera_west" />
+    <material name="blue">
+        <color rgba="0 0 1 1" />
+    </material>
+    <material name="black">
+        <color rgba="0 0 0 1" />
+    </material>
+    <material name="silver">
+        <color rgba="0.79 0.82 0.93 1" />
+    </material>
+    <material name="dark_grey">
+        <color rgba="0.3 0.3 0.3 1" />
+    </material>
 </robot>
